File: Logger/Logger.sch (KiCad schematic (older format))
At the start: 26 parts, among them IC1 ATMEGA328P-A, P1 UART, P2 ISP, P3 microSD_SPI, Q1 SFH309FA-4, Q2 BC817-40, Q3 BC807-40, Y1 16MHz

Commit message: Schaltplan...
Parts:
- removed P1: UART, Pin_Headers:Pin_Header_Straight_1x03_Pitch2.54mm, symbol CONN_01X03
- added D?: LED, symbol LED
- added P1: UART, Pin_Headers:Pin_Header_Straight_1x04_Pitch2.54mm, symbol CONN_01X04
- added R10, R?: 10k, Resistors_SMD:R_0603_HandSoldering, symbol R
- added SW?: SW_SPST_Small, symbol SW_SPST_Small
- C1, C2, C3, C4, C5, C6, C7, C8: footprint Capacitors_SMD:C_0805_HandSoldering -> Capacitors_SMD:C_0603_HandSoldering
- D1, Q1: footprint LEDs:LED-3MM -> LEDs:LED-3MM-SMD
- R1, R2, R3, R4, R5, R6, R7, R8, R9: footprint Resistors_SMD:R_0805_HandSoldering -> Resistors_SMD:R_0603_HandSoldering
Connections:
- net labels added: UART_EN
- wire segments 90 -> 97
Other:
- moved on the sheet: P2

Commit message: Schaltplan Rev A
Parts:
- removed D?: LED, symbol LED
- removed SW?: SW_SPST_Small, symbol SW_SPST_Small
- added R9: 470, Resistors_SMD:R_0603_HandSoldering, symbol R
- added SW1: SW_LED2, symbol SW_LED2
- gave numbers to parts that had none: 1
- renumbered P2 to P1, P1 to P2, R8 to R10, R9 to R12, R10 to R2, R2 to R3, R3 to R4, R4 to R5, R5 to R6, R6 to R7, R7 to R8
Connections:
- net GND: now also SW1.4
- net SW: now reaches IC1.23 ((PCINT8/ADC0)PC0)
- net SW: now also R11.2, SW1.1
- net LED1: now reaches IC1.24 ((PCINT9/ADC1)PC1)
- net LED1: now also R9.1
- net LED2: now reaches IC1.25 ((PCINT10/ADC2)PC2)
- net LED2: now also SW1.2 (K)
- new net: R9.2, SW1.3 (A)
Other:
- note added: "Taster + LED"
- moved on the sheet: R11

Commit message: Schaltplan Rev B
Parts:
- added R6: 10k, Resistors_SMD:R_0805_HandSoldering, symbol R
- C1, C2, C3, C4, C5, C6, C7, C8: footprint Capacitors_SMD:C_0603_HandSoldering -> Capacitors_SMD:C_0805_HandSoldering
- P3: footprint (none) -> Connectors:105162-0101; symbol microSD_SPI -> microSD_SPI_molex
- R1, R2, R3, R4, R5: footprint Resistors_SMD:R_0603_HandSoldering -> Resistors_SMD:R_0805_HandSoldering
- R10: renamed from R9; footprint Resistors_SMD:R_0603_HandSoldering -> Resistors_SMD:R_0805_HandSoldering
- R11: renamed from R10; footprint Resistors_SMD:R_0603_HandSoldering -> Resistors_SMD:R_0805_HandSoldering
- R12: renamed from R11; footprint Resistors_SMD:R_0603_HandSoldering -> Resistors_SMD:R_0805_HandSoldering
- R13: renamed from R12; footprint Resistors_SMD:R_0603_HandSoldering -> Resistors_SMD:R_0805_HandSoldering
- R7: renamed from R6; footprint Resistors_SMD:R_0603_HandSoldering -> Resistors_SMD:R_0805_HandSoldering
- R8: renamed from R7; footprint Resistors_SMD:R_0603_HandSoldering -> Resistors_SMD:R_0805_HandSoldering
- R9: renamed from R8; footprint Resistors_SMD:R_0603_HandSoldering -> Resistors_SMD:R_0805_HandSoldering
- SW1: footprint (none) -> Buttons_Switches_SMD:4FSH9XX
- Y1: footprint Crystals:Crystal_HC49-U_Vertical -> Crystals:SMD_3,2x2,5
Connections:
- net +3V3: now also R6.1
- net GND: now also P3.G1 (SHIELD), P3.G2 (SHIELD), P3.G3 (SHIELD), P3.G4 (SHIELD); no longer P3.10 (SHIELD), P3.11 (SHIELD), P3.12 (SHIELD), P3.9 (SHIELD)
- net UART_EN: now also IC1.26 ((PCINT11/ADC3)PC3); no longer IC1.32 ((PCINT18/INT0)PD2)
- net DETECT: now reaches IC1.27 ((PCINT12/SDA/ADC4)PC4)
- net DETECT: now also P3.9 (DETECET), R6.2
- no-connect marks 0 -> 11
Other:
- moved on the sheet: R10, R12, R7, R8, SW1

Commit message: Schaltplan Rev C and BOM file
Parts:
- C1, C2, C3, C4, C5, C6, C7, C8: footprint Capacitors_SMD:C_0805_HandSoldering -> Capacitors_SMD:C_0603_HandSoldering
- D1: value SFH487-2 -> SFH4356
- R1, R10, R11, R12, R13, R2, R3, R4, R5, R6, R7, R8, R9: footprint Resistors_SMD:R_0805_HandSoldering -> Resistors_SMD:R_0603_HandSoldering
- Y1: footprint Crystals:SMD_3,2x2,5 -> Crystals:SMD_7x4
Changed lines of the file:
@@
 Sheet 1 2
 Title "D0-SD-Logger"
-Date "2017-12-23"
-Rev "B"
+Date "2018-01-07"
+Rev "C"
 Comp "Jonas Gappert"
 Comment1 ""
@@
 F 0 "C4" H 1825 3250 50  0000 L CNN
 F 1 "100n" H 1825 3050 50  0000 L CNN
-F 2 "Capacitors_SMD:C_0805_HandSoldering" H 1838 3000 50  0001 C CNN
+F 2 "Capacitors_SMD:C_0603_HandSoldering" H 1838 3000 50  0001 C CNN
 F 3 "" H 1800 3150 50  0000 C CNN
 	1    1800 3150
@@
 F 0 "C3" H 1425 3250 50  0000 L CNN
 F 1 "100n" H 1425 3050 50  0000 L CNN
-F 2 "Capacitors_SMD:C_0805_HandSoldering" H 1438 3000 50  0001 C CNN
+F 2 "Capacitors_SMD:C_0603_HandSoldering" H 1438 3000 50  0001 C CNN
 F 3 "" H 1400 3150 50  0000 C CNN
 	1    1400 3150
@@
 F 0 "C2" H 1025 3250 50  0000 L CNN
 F 1 "100n" H 1025 3050 50  0000 L CNN
-F 2 "Capacitors_SMD:C_0805_HandSoldering" H 1038 3000 50  0001 C CNN
+F 2 "Capacitors_SMD:C_0603_HandSoldering" H 1038 3000 50  0001 C CNN
 F 3 "" H 1000 3150 50  0000 C CNN
 	1    1000 3150
@@
 F 0 "R3" V 6580 2450 50  0000 C CNN
 F 1 "12k" V 6500 2450 50  0000 C CNN
-F 2 "Resistors_SMD:R_0805_HandSoldering" V 6430 2450 50  0001 C CNN
+F 2 "Resistors_SMD:R_0603_HandSoldering" V 6430 2450 50  0001 C CNN
 F 3 "" H 6500 2450 50  0000 C CNN
 	1    6500 2450
@@
 F 0 "C8" H 7125 1650 50  0000 L CNN
 F 1 "1µ" H 7125 1450 50  0000 L CNN
-F 2 "Capacitors_SMD:C_0805_HandSoldering" H 7138 1400 50  0001 C CNN
+F 2 "Capacitors_SMD:C_0603_HandSoldering" H 7138 1400 50  0001 C CNN
 F 3 "" H 7100 1550 50  0000 C CNN
 	1    7100 1550
@@
 F 0 "R9" V 7680 1550 50  0000 C CNN
 F 1 "12k" V 7600 1550 50  0000 C CNN
-F 2 "Resistors_SMD:R_0805_HandSoldering" V 7530 1550 50  0001 C CNN
+F 2 "Resistors_SMD:R_0603_HandSoldering" V 7530 1550 50  0001 C CNN
 F 3 "" H 7600 1550 50  0000 C CNN
 	1    7600 1550
@@
 P 10200 2000
 F 0 "D1" H 10200 2100 50  0000 C CNN
-F 1 "SFH487-2" H 10200 1900 50  0000 C CNN
+F 1 "SFH4356" H 10200 1900 50  0000 C CNN
 F 2 "LEDs:LED-3MM-SMD" H 10200 2000 50  0001 C CNN
 F 3 "" H 10200 2000 50  0000 C CNN
@@
 F 0 "R13" V 10280 2450 50  0000 C CNN
 F 1 "220" V 10200 2450 50  0000 C CNN
-F 2 "Resistors_SMD:R_0805_HandSoldering" V 10130 2450 50  0001 C CNN
+F 2 "Resistors_SMD:R_0603_HandSoldering" V 10130 2450 50  0001 C CNN
 F 3 "" H 10200 2450 50  0000 C CNN
 	1    10200 2450
@@
 F 0 "R11" V 9630 1500 50  0000 C CNN
 F 1 "12k" V 9550 1500 50  0000 C CNN
-F 2 "Resistors_SMD:R_0805_HandSoldering" V 9480 1500 50  0001 C CNN
+F 2 "Resistors_SMD:R_0603_HandSoldering" V 9480 1500 50  0001 C CNN
 F 3 "" H 9550 1500 50  0000 C CNN
 	1    9550 1500
@@
 F 0 "C5" H 2225 3250 50  0000 L CNN
 F 1 "100n" H 2225 3050 50  0000 L CNN
-F 2 "Capacitors_SMD:C_0805_HandSoldering" H 2238 3000 50  0001 C CNN
+F 2 "Capacitors_SMD:C_0603_HandSoldering" H 2238 3000 50  0001 C CNN
 F 3 "" H 2200 3150 50  0000 C CNN
 	1    2200 3150
@@
 F 0 "C1" H 925 5750 50  0000 L CNN
 F 1 "100n" H 925 5550 50  0000 L CNN
-F 2 "Capacitors_SMD:C_0805_HandSoldering" H 938 5500 50  0001 C CNN
+F 2 "Capacitors_SMD:C_0603_HandSoldering" H 938 5500 50  0001 C CNN
 F 3 "" H 900 5650 50  0000 C CNN
 	1    900  5650
@@
 F 0 "R1" V 980 5150 50  0000 C CNN
 F 1 "10k" V 900 5150 50  0000 C CNN
-F 2 "Resistors_SMD:R_0805_HandSoldering" V 830 5150 50  0001 C CNN
+F 2 "Resistors_SMD:R_0603_HandSoldering" V 830 5150 50  0001 C CNN
 F 3 "" H 900 5150 50  0000 C CNN
 	1    900  5150
@@
 F 0 "Y1" H 2600 5200 50  0000 C CNN
 F 1 "16MHz" H 2600 4900 50  0000 C CNN
-F 2 "Crystals:SMD_3,2x2,5" H 2600 5050 50  0001 C CNN
+F 2 "Crystals:SMD_7x4" H 2600 5050 50  0001 C CNN
 F 3 "" H 2600 5050 50  0000 C CNN
 	1    2600 5050
@@
 F 0 "C7" H 3075 5400 50  0000 L CNN
 F 1 "22p" H 3075 5200 50  0000 L CNN
-F 2 "Capacitors_SMD:C_0805_HandSoldering" H 3088 5150 50  0001 C CNN
+F 2 "Capacitors_SMD:C_0603_HandSoldering" H 3088 5150 50  0001 C CNN
 F 3 "" H 3050 5300 50  0000 C CNN
 	1    3050 5300
@@
 F 0 "C6" H 3075 4900 50  0000 L CNN
 F 1 "22p" H 3075 4700 50  0000 L CNN
-F 2 "Capacitors_SMD:C_0805_HandSoldering" H 3088 4650 50  0001 C CNN
+F 2 "Capacitors_SMD:C_0603_HandSoldering" H 3088 4650 50  0001 C CNN
 F 3 "" H 3050 4800 50  0000 C CNN
 	1    3050 4800
@@
 F 0 "R7" V 7380 4250 50  0000 C CNN
 F 1 "10k" V 7300 4250 50  0000 C CNN
-F 2 "Resistors_SMD:R_0805_HandSoldering" V 7230 4250 50  0001 C CNN
+F 2 "Resistors_SMD:R_0603_HandSoldering" V 7230 4250 50  0001 C CNN
 F 3 "" H 7300 4250 50  0000 C CNN
 	1    7300 4250
@@
 F 0 "R8" V 7580 4250 50  0000 C CNN
 F 1 "10k" V 7500 4250 50  0000 C CNN
-F 2 "Resistors_SMD:R_0805_HandSoldering" V 7430 4250 50  0001 C CNN
+F 2 "Resistors_SMD:R_0603_HandSoldering" V 7430 4250 50  0001 C CNN
 F 3 "" H 7500 4250 50  0000 C CNN
 	1    7500 4250
@@
 F 0 "R5" V 6980 4250 50  0000 C CNN
 F 1 "10k" V 6900 4250 50  0000 C CNN
-F 2 "Resistors_SMD:R_0805_HandSoldering" V 6830 4250 50  0001 C CNN
+F 2 "Resistors_SMD:R_0603_HandSoldering" V 6830 4250 50  0001 C CNN
 F 3 "" H 6900 4250 50  0000 C CNN
 	1    6900 4250
@@
 F 0 "R4" V 6780 4250 50  0000 C CNN
 F 1 "10k" V 6700 4250 50  0000 C CNN
-F 2 "Resistors_SMD:R_0805_HandSoldering" V 6630 4250 50  0001 C CNN
+F 2 "Resistors_SMD:R_0603_HandSoldering" V 6630 4250 50  0001 C CNN
 F 3 "" H 6700 4250 50  0000 C CNN
 	1    6700 4250
@@
 F 0 "R2" V 4580 5150 50  0000 C CNN
 F 1 "10k" V 4500 5150 50  0000 C CNN
-F 2 "Resistors_SMD:R_0805_HandSoldering" V 4430 5150 50  0001 C CNN
+F 2 "Resistors_SMD:R_0603_HandSoldering" V 4430 5150 50  0001 C CNN
 F 3 "" H 4500 5150 50  0000 C CNN
 	1    4500 5150
@@
 F 0 "R12" V 10180 4150 50  0000 C CNN
 F 1 "10k" V 10100 4150 50  0000 C CNN
-F 2 "Resistors_SMD:R_0805_HandSoldering" V 10030 4150 50  0001 C CNN
+F 2 "Resistors_SMD:R_0603_HandSoldering" V 10030 4150 50  0001 C CNN
 F 3 "" H 10100 4150 50  0000 C CNN
 	1    10100 4150
@@
 F 0 "R10" V 9580 4150 50  0000 C CNN
 F 1 "470" V 9500 4150 50  0000 C CNN
-F 2 "Resistors_SMD:R_0805_HandSoldering" V 9430 4150 50  0001 C CNN
+F 2 "Resistors_SMD:R_0603_HandSoldering" V 9430 4150 50  0001 C CNN
 F 3 "" H 9500 4150 50  0000 C CNN
 	1    9500 4150
@@
 F 0 "R6" V 7180 4250 50  0000 C CNN
 F 1 "10k" V 7100 4250 50  0000 C CNN
-F 2 "Resistors_SMD:R_0805_HandSoldering" V 7030 4250 50  0001 C CNN
+F 2 "Resistors_SMD:R_0603_HandSoldering" V 7030 4250 50  0001 C CNN
 F 3 "" H 7100 4250 50  0000 C CNN
 	1    7100 4250
