File: Logger/Power.sch (KiCad schematic (older format))
At the start: 5 parts, among them P4 Vin, U1 78M33C

Commit message: Schaltplan...
Parts:
- C10, C9: footprint Capacitors_SMD:C_0805_HandSoldering -> Capacitors_SMD:C_0603_HandSoldering
Changed lines of the file:
@@
 EESchema Schematic File Version 2
+LIBS:Logger-rescue
 LIBS:power
 LIBS:device
@@
 F 0 "C10" H 7825 3450 50  0000 L CNN
 F 1 "1µ" H 7825 3250 50  0000 L CNN
-F 2 "Capacitors_SMD:C_0805_HandSoldering" H 7838 3200 50  0001 C CNN
+F 2 "Capacitors_SMD:C_0603_HandSoldering" H 7838 3200 50  0001 C CNN
 F 3 "" H 7800 3350 50  0000 C CNN
 	1    7800 3350
@@
 F 0 "C9" H 6625 3450 50  0000 L CNN
 F 1 "2µ2" H 6625 3250 50  0000 L CNN
-F 2 "Capacitors_SMD:C_0805_HandSoldering" H 6638 3200 50  0001 C CNN
+F 2 "Capacitors_SMD:C_0603_HandSoldering" H 6638 3200 50  0001 C CNN
 F 3 "" H 6600 3350 50  0000 C CNN
 	1    6600 3350
@@
 $EndComp
 $Comp
-L GND #PWR25
+L GND #PWR022
 U 1 1 5A289237
 P 7200 3600
-F 0 "#PWR25" H 7200 3350 50  0001 C CNN
+F 0 "#PWR022" H 7200 3350 50  0001 C CNN
 F 1 "GND" H 7200 3450 50  0000 C CNN
 F 2 "" H 7200 3600 50  0000 C CNN
@@
 $EndComp
 $Comp
-L GND #PWR27
+L GND #PWR023
 U 1 1 5A28923D
 P 7800 3600
-F 0 "#PWR27" H 7800 3350 50  0001 C CNN
+F 0 "#PWR023" H 7800 3350 50  0001 C CNN
 F 1 "GND" H 7800 3450 50  0000 C CNN
 F 2 "" H 7800 3600 50  0000 C CNN
@@
 $EndComp
 $Comp
-L +3V3 #PWR26
+L +3V3 #PWR024
 U 1 1 5A289243
 P 7800 2900
-F 0 "#PWR26" H 7800 2750 50  0001 C CNN
+F 0 "#PWR024" H 7800 2750 50  0001 C CNN
 F 1 "+3V3" H 7800 3040 50  0000 C CNN
 F 2 "" H 7800 2900 50  0000 C CNN
@@
 $EndComp
 $Comp
-L VCC #PWR23
+L VCC #PWR025
 U 1 1 5A289249
 P 6600 2900
-F 0 "#PWR23" H 6600 2750 50  0001 C CNN
+F 0 "#PWR025" H 6600 2750 50  0001 C CNN
 F 1 "VCC" H 6600 3050 50  0000 C CNN
 F 2 "" H 6600 2900 50  0000 C CNN
@@
 $EndComp
 $Comp
-L GND #PWR21
+L GND #PWR026
 U 1 1 5A28925D
 P 4500 3400
-F 0 "#PWR21" H 4500 3150 50  0001 C CNN
+F 0 "#PWR026" H 4500 3150 50  0001 C CNN
 F 1 "GND" H 4500 3250 50  0000 C CNN
 F 2 "" H 4500 3400 50  0000 C CNN
@@
 $EndComp
 $Comp
-L VCC #PWR22
+L VCC #PWR027
 U 1 1 5A289263
 P 5800 2900
-F 0 "#PWR22" H 5800 2750 50  0001 C CNN
+F 0 "#PWR027" H 5800 2750 50  0001 C CNN
 F 1 "VCC" H 5800 3050 50  0000 C CNN
 F 2 "" H 5800 2900 50  0000 C CNN
@@
 $EndComp
 $Comp
-L GND #PWR24
+L GND #PWR028
 U 1 1 5A289270
 P 6600 3600
-F 0 "#PWR24" H 6600 3350 50  0001 C CNN
+F 0 "#PWR028" H 6600 3350 50  0001 C CNN
 F 1 "GND" H 6600 3450 50  0000 C CNN
 F 2 "" H 6600 3600 50  0000 C CNN

Commit message: Schaltplan Rev B
Parts:
- C10, C9: footprint Capacitors_SMD:C_0603_HandSoldering -> Capacitors_SMD:C_0805_HandSoldering
- D2: footprint (none) -> Housings_SOIC:SOIC-4
Changed lines of the file:
@@
 encoding utf-8
 Sheet 2 2
-Title ""
-Date ""
-Rev ""
+Title "D0-SD-Logger"
+Date "2017-12-23"
+Rev "B"
 Comp "Jonas Gappert"
 Comment1 ""
@@
 F 0 "C10" H 7825 3450 50  0000 L CNN
 F 1 "1µ" H 7825 3250 50  0000 L CNN
-F 2 "Capacitors_SMD:C_0603_HandSoldering" H 7838 3200 50  0001 C CNN
+F 2 "Capacitors_SMD:C_0805_HandSoldering" H 7838 3200 50  0001 C CNN
 F 3 "" H 7800 3350 50  0000 C CNN
 	1    7800 3350
@@
 F 0 "C9" H 6625 3450 50  0000 L CNN
 F 1 "2µ2" H 6625 3250 50  0000 L CNN
-F 2 "Capacitors_SMD:C_0603_HandSoldering" H 6638 3200 50  0001 C CNN
+F 2 "Capacitors_SMD:C_0805_HandSoldering" H 6638 3200 50  0001 C CNN
 F 3 "" H 6600 3350 50  0000 C CNN
 	1    6600 3350
@@
 $EndComp
 $Comp
-L GND #PWR28
+L GND #PWR024
 U 1 1 5A289237
 P 7200 3600
-F 0 "#PWR28" H 7200 3350 50  0001 C CNN
+F 0 "#PWR024" H 7200 3350 50  0001 C CNN
 F 1 "GND" H 7200 3450 50  0000 C CNN
 F 2 "" H 7200 3600 50  0000 C CNN
@@
 $EndComp
 $Comp
-L GND #PWR30
+L GND #PWR025
 U 1 1 5A28923D
 P 7800 3600
-F 0 "#PWR30" H 7800 3350 50  0001 C CNN
+F 0 "#PWR025" H 7800 3350 50  0001 C CNN
 F 1 "GND" H 7800 3450 50  0000 C CNN
 F 2 "" H 7800 3600 50  0000 C CNN
@@
 $EndComp
 $Comp
-L +3V3 #PWR29
+L +3V3 #PWR026
 U 1 1 5A289243
 P 7800 2900
-F 0 "#PWR29" H 7800 2750 50  0001 C CNN
+F 0 "#PWR026" H 7800 2750 50  0001 C CNN
 F 1 "+3V3" H 7800 3040 50  0000 C CNN
 F 2 "" H 7800 2900 50  0000 C CNN
@@
 $EndComp
 $Comp
-L VCC #PWR26
+L VCC #PWR027
 U 1 1 5A289249
 P 6600 2900
-F 0 "#PWR26" H 6600 2750 50  0001 C CNN
+F 0 "#PWR027" H 6600 2750 50  0001 C CNN
 F 1 "VCC" H 6600 3050 50  0000 C CNN
 F 2 "" H 6600 2900 50  0000 C CNN
@@
 F 0 "D2" H 5300 3500 50  0000 L CNN
 F 1 "D_BRIDGE" H 5300 3400 50  0000 L CNN
-F 2 "" H 5000 3200 50  0001 C CNN
+F 2 "Housings_SOIC:SOIC-4" H 5000 3200 50  0001 C CNN
 F 3 "" H 5000 3200 50  0000 C CNN
 	1    5000 3200
@@
 $EndComp
 $Comp
-L GND #PWR24
+L GND #PWR028
 U 1 1 5A28925D
 P 4500 3400
-F 0 "#PWR24" H 4500 3150 50  0001 C CNN
+F 0 "#PWR028" H 4500 3150 50  0001 C CNN
 F 1 "GND" H 4500 3250 50  0000 C CNN
 F 2 "" H 4500 3400 50  0000 C CNN
@@
 $EndComp
 $Comp
-L VCC #PWR25
+L VCC #PWR029
 U 1 1 5A289263
 P 5800 2900
-F 0 "#PWR25" H 5800 2750 50  0001 C CNN
+F 0 "#PWR029" H 5800 2750 50  0001 C CNN
 F 1 "VCC" H 5800 3050 50  0000 C CNN
 F 2 "" H 5800 2900 50  0000 C CNN
@@
 $EndComp
 $Comp
-L GND #PWR27
+L GND #PWR030
 U 1 1 5A289270
 P 6600 3600
-F 0 "#PWR27" H 6600 3350 50  0001 C CNN
+F 0 "#PWR030" H 6600 3350 50  0001 C CNN
 F 1 "GND" H 6600 3450 50  0000 C CNN
 F 2 "" H 6600 3600 50  0000 C CNN

Commit message: Schaltplan Rev C and BOM file
Parts:
- C10, C9: footprint Capacitors_SMD:C_0805_HandSoldering -> Capacitors_SMD:C_0603_HandSoldering
Changed lines of the file:
@@
 Sheet 2 2
 Title "D0-SD-Logger"
-Date "2017-12-23"
-Rev "B"
+Date "2018-01-07"
+Rev "C"
 Comp "Jonas Gappert"
 Comment1 ""
@@
 F 0 "C10" H 7825 3450 50  0000 L CNN
 F 1 "1µ" H 7825 3250 50  0000 L CNN
-F 2 "Capacitors_SMD:C_0805_HandSoldering" H 7838 3200 50  0001 C CNN
+F 2 "Capacitors_SMD:C_0603_HandSoldering" H 7838 3200 50  0001 C CNN
 F 3 "" H 7800 3350 50  0000 C CNN
 	1    7800 3350
@@
 F 0 "C9" H 6625 3450 50  0000 L CNN
 F 1 "2µ2" H 6625 3250 50  0000 L CNN
-F 2 "Capacitors_SMD:C_0805_HandSoldering" H 6638 3200 50  0001 C CNN
+F 2 "Capacitors_SMD:C_0603_HandSoldering" H 6638 3200 50  0001 C CNN
 F 3 "" H 6600 3350 50  0000 C CNN
 	1    6600 3350

Commit message: Schaltplan Rev D, Gleichrichter geaendert
Parts:
- D2: symbol D_BRIDGE -> D_BRIDGE_2
Connections:
- net GND: now also D2.2 (-); no longer D2.1 (-)
- net VCC: now also D2.1 (+); no longer D2.3 (+)
- net at P4.2 (P2): now also D2.3; no longer D2.2
Changed lines of the file:
@@
 Sheet 2 2
 Title "D0-SD-Logger"
-Date "2018-01-07"
-Rev "C"
+Date "2018-01-19"
+Rev "D"
 Comp "Jonas Gappert"
 Comment1 ""
@@
 $EndComp
 $Comp
-L D_BRIDGE D2
+L D_BRIDGE_2 D2
 U 1 1 5A28924F
 P 5000 3200
