File: Logger/Logger.kicad_pcb (KiCad board)
At the start: 2 copper layers, 27 x 27 mm, 29 parts, among them IC1 ATMEGA328P-A, P1 UART, P2 ISP, P4 Vin, Q1 SFH309FA-4, Q2 BC817-40, Q3 BC807-40, U1 78M33C, Y1 16MHz

Commit message: Schaltplan...
Parts:
- added R10: 10k, Resistors_SMD:R_0603_HandSoldering, B.Cu at (101.1, 113.7)
- C1, C10, C2, C3, C4, C5, C6, C7, C8, C9: footprint Capacitors_SMD:C_0805_HandSoldering -> Capacitors_SMD:C_0603_HandSoldering; moved to B.Cu
- D1, Q1: footprint LEDs:LED-3MM -> LEDs:LED-3MM-SMD; moved to B.Cu
- P1: footprint Pin_Headers:Pin_Header_Straight_1x03_Pitch2.54mm -> Pin_Headers:Pin_Header_Straight_1x04_Pitch2.54mm
- Q2, Q3: moved to B.Cu
- R1, R2, R3, R4, R5, R6, R7, R8, R9: footprint Resistors_SMD:R_0805_HandSoldering -> Resistors_SMD:R_0603_HandSoldering; moved to B.Cu
- moved P4 125.1 mm to (98.6, 118.7)
- moved C10 116.2 mm to (115.1, 130.2)
- moved C9 113.7 mm to (118.9, 113.7), turned to 90 degrees
- moved Q2 91.0 mm to (99.8, 125.1)
- moved R8 90.2 mm to (115.1, 116.2)
- moved C1 90.2 mm to (104.9, 116.2)
- moved C8 90.1 mm to (110.0, 116.2)
- moved U1 89.6 mm to (126.5, 110.9), turned to 270 degrees
- moved R3 88.8 mm to (115.1, 113.7)
- moved R7 88.7 mm to (110.0, 113.7)
- moved C5 88.6 mm to (104.9, 113.7)
- moved C4 80.0 mm to (104.9, 111.1)
- moved R2 79.8 mm to (115.1, 111.1)
- moved R4 79.7 mm to (110.0, 111.1)
- moved R5 75.7 mm to (115.1, 127.6)
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Connections:
- IC1 pad 32: Net-(IC1-Pad32) -> UART_EN
- P1 pad 1: RX -> UART_EN
- P1 pad 2: TX -> RX
- P1 pad 3: GND -> TX
- Q1 pad 1: Net-(Q1-Pad1) -> +3V3
- Q1 pad 2: (no net) -> Net-(Q1-Pad2)
- Q2 pad 1: Net-(Q1-Pad1) -> Net-(Q1-Pad2)
- R2 pad 1: Net-(Q1-Pad1) -> Net-(Q1-Pad2)

Commit message: Schaltplan Rev B
Parts:
- added D2: D_BRIDGE, Housings_SOIC:SOIC-4, F.Cu at (153.9, 103.9)
- added P3: microSD_SPI, Connectors:105162-0101, F.Cu at (145.0, 81.7)
- added R11: 12k, Resistors_SMD:R_0805_HandSoldering, B.Cu at (151.2, 88.7)
- added R12: 10k, Resistors_SMD:R_0805_HandSoldering, B.Cu at (147.4, 84.8)
- added R13: 220, Resistors_SMD:R_0805_HandSoldering, B.Cu at (142.5, 89.9)
- added SW1: SW_LED2, Buttons_Switches_SMD:4FSH9XX, F.Cu at (151.2, 91.2)
- C1, C2, C3, C4, C5, C6, C7, C8: footprint Capacitors_SMD:C_0603_HandSoldering -> Capacitors_SMD:C_0805_HandSoldering
- C10, C9: footprint Capacitors_SMD:C_0603_HandSoldering -> Capacitors_SMD:C_0805_HandSoldering; moved to F.Cu
- IC1: moved to B.Cu
- P1: value UART -> ISP; footprint Pin_Headers:Pin_Header_Straight_1x04_Pitch2.54mm -> Pin_Headers:Pin_Header_Straight_2x03_Pitch2.54mm
- P2: value ISP -> UART; footprint Pin_Headers:Pin_Header_Straight_2x03_Pitch2.54mm -> Pin_Headers:Pin_Header_Straight_1x04_Pitch2.54mm
- R1, R4, R5, R6: footprint Resistors_SMD:R_0603_HandSoldering -> Resistors_SMD:R_0805_HandSoldering
- R10: value 10k -> 470; footprint Resistors_SMD:R_0603_HandSoldering -> Resistors_SMD:R_0805_HandSoldering
- R2, R7, R8: value 12k -> 10k; footprint Resistors_SMD:R_0603_HandSoldering -> Resistors_SMD:R_0805_HandSoldering
- R3: value 10k -> 12k; footprint Resistors_SMD:R_0603_HandSoldering -> Resistors_SMD:R_0805_HandSoldering
- R9: value 220 -> 12k; footprint Resistors_SMD:R_0603_HandSoldering -> Resistors_SMD:R_0805_HandSoldering
- Y1: footprint Crystals:Crystal_HC49-U_Vertical -> Crystals:SMD_3,2x2,5; moved to B.Cu
- moved P4 60.0 mm to (155.2, 98.8)
- moved C7 56.9 mm to (147.5, 89.9)
- moved R6 56.8 mm to (147.4, 87.4)
- moved R10 55.9 mm to (147.4, 82.3), turned to 0 degrees
- moved R1 53.6 mm to (142.3, 82.3)
- moved Q2 53.5 mm to (142.5, 92.7)
- moved C3 53.4 mm to (147.5, 92.1)
- moved P2 52.4 mm to (155.2, 87.4), turned to 0 degrees
- moved R7 51.0 mm to (151.2, 83.6)
- moved Y1 49.7 mm to (150.1, 103.9)
- moved C5 49.3 mm to (152.3, 100.1)
- moved C4 49.0 mm to (152.3, 98.8)
- moved C6 48.7 mm to (142.5, 84.8)
- moved R5 48.6 mm to (142.3, 87.4)
- moved R4 48.2 mm to (151.2, 86.1)
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Connections:
- IC1 pad 23: Net-(IC1-Pad23) -> SW
- IC1 pad 24: Net-(IC1-Pad24) -> LED1
- IC1 pad 25: Net-(IC1-Pad25) -> LED2
- IC1 pad 26: Net-(IC1-Pad26) -> UART_EN
- IC1 pad 27: Net-(IC1-Pad27) -> DETECT
- IC1 pad 32: UART_EN -> Net-(IC1-Pad32)
- P1 pad 1: UART_EN -> MISO
- P1 pad 2: RX -> +3V3
- P1 pad 3: TX -> SCK
- P1 pad 4: GND -> MOSI
- P2 pad 1: MISO -> UART_EN
- P2 pad 2: +3V3 -> RX
- P2 pad 3: SCK -> TX
- P2 pad 4: MOSI -> GND
- R10 pad 1: +3V3 -> LED1
- R10 pad 2: UART_EN -> Net-(R10-Pad2)
- R2 pad 1: Net-(Q1-Pad2) -> +3V3
- R2 pad 2: GND -> UART_EN
- R3 pad 1: +3V3 -> Net-(Q1-Pad2)
- R3 pad 2: MISO -> GND
- R4 pad 2: SS -> MISO
- R5 pad 2: Net-(P3-Pad8) -> SS
- R6 pad 2: Net-(P3-Pad1) -> DETECT
- R7 pad 2: RX -> Net-(P3-Pad8)
- R8 pad 1: Net-(Q3-Pad1) -> +3V3
- R8 pad 2: TX -> Net-(P3-Pad1)
- R9 pad 1: Net-(D1-Pad1) -> +3V3
- R9 pad 2: GND -> RX
Other:
- board size 27 x 27 mm -> 29 x 29 mm
- rule pad_to_mask_clearance: 0.2 -> 0

Commit message: Schaltplan Rev C and BOM file
Parts:
- C1, C10, C2, C3, C4, C5, C6, C7, C8, C9: footprint Capacitors_SMD:C_0805_HandSoldering -> Capacitors_SMD:C_0603_HandSoldering
- D1: value SFH487-2 -> SFH4356
- R1, R10, R11, R12, R13, R2, R3, R4, R5, R6, R7, R8, R9: footprint Resistors_SMD:R_0805_HandSoldering -> Resistors_SMD:R_0603_HandSoldering
- Y1: footprint Crystals:SMD_3,2x2,5 -> Crystals:SMD_7x4
- moved R9 78.2 mm to (214.0, 96.0)
- moved R8 72.9 mm to (208.9, 102.3)
- moved R2 66.7 mm to (201.3, 89.8)
- moved R7 65.7 mm to (214.2, 102.3)
- moved R1 64.1 mm to (206.4, 83.5)
- moved R6 63.7 mm to (207.4, 108.5)
- moved R13 62.5 mm to (203.7, 102.3)
- moved R12 62.4 mm to (208.7, 96.0)
- moved C8 61.9 mm to (211.5, 83.5)
- moved R10 60.8 mm to (202.2, 108.5)
- moved C1 57.7 mm to (193.5, 101.9)
- moved R4 55.5 mm to (206.6, 89.8)
- moved R3 52.4 mm to (186.6, 108.2)
- moved C5 51.5 mm to (203.6, 96.0)
- moved R11 49.9 mm to (196.9, 108.5)
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
Commit message: PCB save
Parts:
- C10, C9, D2, U1: moved to B.Cu
- moved C9 26.9 mm to (155.2, 78.5)
- moved C10 14.0 mm to (136.7, 87.4)
- moved U1 12.7 mm to (143.7, 91.8), turned to 180 degrees
- moved D2 11.1 mm to (150.1, 88.1), turned to 0 degrees
- moved C2 2.84 mm to (128.5, 102.0)
- moved P2 2.54 mm to (153.9, 87.4)
- moved P4 2.54 mm to (156.4, 95.0)
- moved P1 1.27 mm to (133.6, 91.2)
Connections:
- D2 pad 1: GND -> VCC
- D2 pad 2: Net-(D2-Pad2) -> GND
- D2 pad 3: VCC -> Net-(D2-Pad3)
- P4 pad 2: Net-(D2-Pad2) -> Net-(D2-Pad3)

Commit message: PCB Save
Parts:
- C1, R1, Y1: moved to F.Cu
- moved R1 70.4 mm to (141.8, 111.5)
- moved C1 47.4 mm to (146.9, 110.9)
- moved C3 9.65 mm to (137.4, 101.8)
- moved C2 9.02 mm to (137.4, 103.4)
- moved C9 8.08 mm to (149.4, 84.2), turned to 0 degrees
- moved Y1 7.22 mm to (144.6, 102.6), turned to 0 degrees
- moved C10 4.58 mm to (139.3, 91.2), turned to 90 degrees
- moved C6 4.45 mm to (137.4, 100.2), turned to 0 degrees
- moved IC1 2.86 mm to (145.0, 102.2)
- moved P4 2.54 mm to (156.4, 92.5), turned to 0 degrees
- moved C7 2.40 mm to (137.4, 98.6), turned to 0 degrees
- moved D2 1.27 mm to (150.1, 89.4)
- moved U1 0.38 mm to (143.7, 92.2)
Routing:
- net GND: track 0.00 -> 11.3 mm
- net Net-(D2-Pad4): track 0.00 -> 10.1 mm
- net VCC: track 0.00 -> 9.29 mm
- net Net-(D2-Pad3): track 0.00 -> 6.07 mm
Other:
- net class Default: clearance 0.2 -> 0.254; trace_width 0.25 -> 0.3048; via_dia 0.6 -> 0.6096; via_drill 0.4 -> 0.3048
- rule trace_clearance: 0.2 -> 0.254
- rule trace_min: 0.2 -> 0.2032
- rule via_min_drill: 0.3 -> 0.3048
- rule via_min_size: 0.4 -> 0.6096
